File: PCB's/MacroPad/MacroPad.kicad_pcb (KiCad board)
At the start: 2 copper layers, 144 x 79 mm, 59 parts, among them SW1 SW_Push, SW2 SW_Push, SW3 SW_Push, SW4 SW_Push, SW5 SW_Push, SW6 SW_Push

Commit message: Add current JLCPCB BOM and placement files
Parts:
- S1, S2: value EVQ-Q2B03W -> EVQ-Q2K03W
Changed lines of the file:
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@@
 			)
 		)
-		(property "Value" "EVQ-Q2B03W"
+		(property "Value" "EVQ-Q2K03W"
 			(at 0.033211 3.745233 0)
 			(layer "F.Fab")
@@
 			)
 		)
-		(property "Value" "EVQ-Q2B03W"
+		(property "Value" "EVQ-Q2K03W"
 			(at 0.033211 3.745233 0)
 			(layer "F.Fab")
