File: PCB's/MacroPad/MacroPad.kicad_sch (KiCad schematic)
At the start: 59 parts, among them SW1 SW_Push, SW2 SW_Push, SW3 SW_Push, SW4 SW_Push, SW5 SW_Push, SW6 SW_Push

Commit message: Add current JLCPCB BOM and placement files
Parts:
- S1, S2: value EVQ-Q2B02W -> EVQ-Q2K03W
Changed lines of the file:
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@@
 			)
 		)
-		(property "Value" "EVQ-Q2B02W"
+		(property "Value" "EVQ-Q2K03W"
 			(at 208.28 102.87 0)
 			(effects
@@
 			)
 		)
-		(property "Value" "EVQ-Q2B02W"
+		(property "Value" "EVQ-Q2K03W"
 			(at 208.28 83.82 0)
 			(effects
